File: StartStopTascam.kicad_pcb (KiCad board)
At the start: 2 copper layers, 69.1 x 53.8 mm, 15 parts, among them J1 Jack_LJB0670, J2 Jack_LJB0670, J3 DB9_Male, P1 CONN_02X03, U1 MAX232

Commit message: kicad
Parts:
- added C3: 10U-X5R_25V#1210, D&R_Passive:C_1210, B.Cu at (89.6, 69.8)
- added C4: 10U-X5R_25V#1210, D&R_Passive:C_1210, B.Cu at (83.4, 69.8)
- added R3: 4k7, D&R_Passive:C_0603, B.Cu at (107.2, 55.4)
- added R4: 4k7, D&R_Passive:C_0603, B.Cu at (107.2, 58.7)
- C5, C7: value 10U-ALU_16V#CASE_B -> 10U-X5R_25V#1210; footprint D&R_Passive:C_0805 -> D&R_Passive:C_1210
- C8, C9: value 10U-ALU_16V#CASE_B -> 100N-X7R_50V#0603-D&R_Passive; footprint D&R_Passive:C_0805 -> D&R_Passive:C_0603
- J1, J2: value Jack_LJB0670 -> Jack_Stack_LJB0671; footprint D&R_Conn:LJB0670 -> D&R_Conn:LJB0671-12
- moved C9 33.7 mm to (110.7, 58.7), turned to 180 degrees
- moved C1 27.0 mm to (72.1, 54.5), turned to 0 degrees
- moved C8 26.1 mm to (110.7, 55.4), turned to 180 degrees
- moved R1 23.6 mm to (75.4, 54.5)
- moved J1 22.9 mm to (86.4, 38.5)
- moved J2 22.9 mm to (109.2, 38.5)
- moved C2 6.81 mm to (72.1, 58.7), turned to 0 degrees
- moved R2 3.64 mm to (75.4, 58.7)
- moved C7 0.81 mm to (83.3, 63.2), turned to 0 degrees
- moved C5 0.65 mm to (89.4, 63.2)
Connections:
- C1 pad 1: GND -> /GND
- C2 pad 1: GND -> /GND
- C5 pad 1: Net-(C5-Pad1) -> VCC
- C5 pad 2: Net-(C5-Pad2) -> /Net-(U1-Pad2)
- C6 pad 2: GND -> /GND
- C7 pad 1: Net-(C7-Pad1) -> /Net-(U1-Pad6)
- C7 pad 2: Net-(C7-Pad2) -> /GND
- C8 pad 1: Net-(C8-Pad1) -> /GND
- C8 pad 2: VCC -> /Net-(XA1-PadA0)
- C9 pad 1: GND -> /GND
- C9 pad 2: Net-(C9-Pad2) -> /Net-(XA1-PadA1)
- J1 pad 1: Net-(J1-Pad1) -> /Net-(R2-Pad1)
- J1 pad 3: GND -> /Net-(R1-Pad1)
- J1 pad 5: unconnected-(J1-Pad5) -> /GND
- J2 pad 3: GND -> Net-(J2-Pad3)
- J2 pad 5: unconnected-(J2-Pad5) -> /GND
- J3 pad 0: GND -> (no net)
- J3 pad 5: GND -> /GND
- R1 pad 1: Net-(J1-Pad1) -> /Net-(R1-Pad1)
- R2 pad 1: Net-(J2-Pad1) -> /Net-(R2-Pad1)
- U1 pad 1: Net-(C5-Pad1) -> /Net-(U1-Pad1)
- U1 pad 15: GND -> /GND
- U1 pad 2: Net-(C8-Pad1) -> /Net-(U1-Pad2)
- U1 pad 3: Net-(C5-Pad2) -> /Net-(U1-Pad3)
- U1 pad 4: Net-(C7-Pad1) -> /Net-(U1-Pad4)
- U1 pad 5: Net-(C7-Pad2) -> /Net-(U1-Pad5)
- U1 pad 6: Net-(C9-Pad2) -> /Net-(U1-Pad6)
- XA1 pad A0: unconnected-(XA1-PadA0) -> /Net-(XA1-PadA0)
- XA1 pad A1: unconnected-(XA1-PadA1) -> /Net-(XA1-PadA1)
- XA1 pad GND3: GND -> /GND
Routing:
- net /Net-(XA1-PadA1): track 0.00 -> 52.8 mm
- net /Net-(XA1-PadA0): track 0.00 -> 43.3 mm
- net /Net-(XA1-PadA2): track 37.6 -> 22.9 mm
- net /Net-(XA1-PadA3): track 21.3 -> 30.2 mm
- net /Net-(U1-Pad6): track 0.00 -> 5.49 mm
- net /GND: track 0.00 -> 4.89 mm, vias 0 -> 1
- net /Net-(R1-Pad1): track 0.00 -> 4.61 mm
- net /Net-(U1-Pad3): track 0.00 -> 4.33 mm
- net Net-(C5-Pad2): track 4.19 -> 0.00 mm
- net /Net-(U1-Pad4): track 0.00 -> 3.91 mm
- net /Net-(U1-Pad1): track 0.00 -> 3.82 mm
- net /Net-(U1-Pad5): track 0.00 -> 3.72 mm
- net /Net-(U1-Pad2): track 0.00 -> 3.56 mm
- net /Net-(R2-Pad1): track 0.00 -> 3.52 mm
- net Net-(J1-Pad1): track 3.48 -> 0.00 mm
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- added copper zone on B.Cu, net /GND
- added copper zone on F.Cu, net /GND
- removed copper zone on B.Cu, net GND
- removed copper zone on F.Cu, net GND

Commit message: kicad
Connections:
- XA1 pad GND2: unconnected-(XA1-PadGND2) -> /GND
Routing:
- net /GND: track 4.89 -> 7.43 mm
Other:
- board size 69.1 x 53.8 mm -> 68.6 x 53.3 mm

Commit message: Kicad
Kicad
Parts:
- added D1: TSAL4400, LED_THT:LED_D3.0mm_IRBlack, F.Cu at (75.7, 78.7)
- added R5: 470R#0603, D&R_Passive:R_0603, B.Cu at (75.4, 71.6)
- moved C3 0.91 mm to (88.6, 69.8)
- moved J1 0.89 mm to (86.4, 37.6)
- moved J2 0.89 mm to (109.2, 37.6)
- moved C4 0.89 mm to (82.5, 69.8)
- moved C2 0.76 mm to (72.1, 57.9)
- moved C8 0.76 mm to (110.7, 54.6)
- moved C9 0.76 mm to (110.7, 57.9)
- moved R2 0.76 mm to (75.4, 57.9)
- moved R3 0.76 mm to (107.2, 54.6)
- moved R4 0.76 mm to (107.2, 57.9)
- moved U1 0.27 mm to (91.4, 66.3)
- moved C1 0.13 mm to (72.1, 54.6)
- moved R1 0.13 mm to (75.4, 54.6)
Connections:
- XA1 pad D2: unconnected-(XA1-PadD2) -> Net-(XA1-PadD2)
- XA1 pad D3: unconnected-(XA1-PadD3) -> Net-(U1-Pad11)
- XA1 pad D4: Net-(U1-Pad11) -> Net-(U1-Pad12)
- XA1 pad D5: Net-(U1-Pad12) -> unconnected-(XA1-PadD5)
Routing:
- net VCC: track 50.8 -> 64.1 mm
- net Net-(D1-Pad2): track 0.00 -> 10.4 mm
- net Net-(XA1-PadD2): track 0.00 -> 5.29 mm
- net /Net-(XA1-PadA1): track 52.8 -> 53.8 mm
- net Net-(U1-Pad11): track 10.9 -> 10.0 mm
- net Net-(U1-Pad12): track 10.9 -> 10.0 mm
- net /Net-(XA1-PadA0): track 43.3 -> 42.5 mm
- net /Net-(XA1-PadA3): track 30.2 -> 29.5 mm
- net /GND: track 7.43 -> 7.66 mm, vias 1 -> 9
