File: StartStopTascam.kicad_sch (KiCad schematic)
At the start: 19 parts, among them J1 Jack_LJB0670, J2 Jack_LJB0670, J3 DB9_Male, P1 CONN_02X03, U1 MAX232

Commit message: kicad
Parts:
- removed C2, C4: (no value), symbol StartStopTascam-rescue:100N-X7R_50V#0603-D&R_Passive
- removed R2, R4: (no value), D&R_Passive:C_0603, symbol StartStopTascam-rescue:R-D&R_Passive
- C5, C7, C8, C9: value 10U-ALU_16V#CASE_B -> (none); footprint D&R_Passive:C_0805 -> (none)
- C6: value 100N-X7R_50V#0603 -> (none); footprint D&R_Passive:C_0603 -> (none)
- J1, J2: value Jack_LJB0670 -> (none); footprint D&R_Conn:LJB0670 -> (none)
- J3: value DB9_Male -> (none); footprint Connector_Dsub:DSUB-9_Male_Horizontal_P2.77x2.84mm_EdgePinOffset4.94mm_Housed_MountingHolesOffset7.48mm -> (none)
- P1: value CONN_02X03 -> (none); footprint D&R_Conn:HEADER_2x3P -> (none)
- R1: footprint D&R_Passive:C_0603 -> (none)
- R2: renamed from R3; footprint D&R_Passive:C_0603 -> (none)
- U1: value MAX232 -> (none); footprint Package_DIP:DIP-16_W7.62mm -> (none)
- XA1: value Arduino_Uno_Shield -> (none); footprint Arduino:Arduino_Uno_Shield_Hat -> (none)
- renumbered C3 to C2
Connections:
- net GND: now also J1.3 (R), J2.3 (R); no longer J1.5 (S), J2.5 (S)
- net at U1.11 (T1IN): now also XA1.D10 (D10_CS); no longer XA1.MOSI (SPI_MOSI)
- net at U1.12 (R1OUT): now also XA1.D11; no longer XA1.MISO (SPI_MISO)
- net at C2.2, R2.2: now also XA1.A3; no longer XA1.A1
- net at XA1.A2: now also C1.2, R1.2
- no-connect marks 43 -> 48
Other:
- moved on the sheet: C1, C2

Commit message: kicad
Parts:
- C1, C2: value (none) -> 100N-X7R_50V#0603-D&R_Passive; footprint (none) -> D&R_Passive:C_0603
- C5, C7, C8, C9: value (none) -> 10U-ALU_16V#CASE_B; footprint (none) -> D&R_Passive:C_0805
- C6: value (none) -> 100N-X7R_50V#0603; footprint (none) -> D&R_Passive:C_0603
- J1, J2: value (none) -> Jack_LJB0670; footprint (none) -> D&R_Conn:LJB0670
- J3: value (none) -> DB9_Male; footprint (none) -> Connector_Dsub:DSUB-9_Male_Horizontal_P2.77x2.84mm_EdgePinOffset4.94mm_Housed_MountingHolesOffset7.48mm
- P1: value (none) -> CONN_02X03; footprint (none) -> D&R_Conn:HEADER_2x3P
- R1, R2: value (none) -> 4k7; footprint (none) -> D&R_Passive:C_0603
- U1: value (none) -> MAX232; footprint (none) -> Package_DIP:DIP-16_W7.62mm
- XA1: value (none) -> Arduino_Uno_Shield; footprint (none) -> Arduino:Arduino_Uno_Shield_Hat
Connections:
- net at U1.11 (T1IN): now also XA1.D4; no longer XA1.D10 (D10_CS)
- net at U1.12 (R1OUT): now also XA1.D5; no longer XA1.D11
Changed lines of the file:
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@@
   (no_connect (at 94.615 115.57))
   (no_connect (at 94.615 110.49))
-  (no_connect (at 160.655 74.93))
   (no_connect (at 94.615 107.95))
   (no_connect (at 160.655 107.95))
   (no_connect (at 160.655 110.49))
   (no_connect (at 94.615 67.31))
-  (no_connect (at 160.655 72.39))
   (no_connect (at 47.625 76.2))
   (no_connect (at 47.625 118.745))
@@
   (no_connect (at 160.655 100.33))
   (no_connect (at 160.655 102.87))
+  (no_connect (at 160.655 87.63))
+  (no_connect (at 160.655 90.17))
   (wire (pts (xy 261.62 125.73) (xy 261.62 120.65))
     (stroke (width 0) (type default) (color 0 0 0 0))
   )
+  (wire (pts (xy 167.005 74.93) (xy 167.005 107.95))
+    (stroke (width 0) (type default) (color 0 0 0 0))
+  )
   (wire (pts (xy 229.87 138.43) (xy 249.555 138.43))
     (stroke (width 0) (type default) (color 0 0 0 0))
@@
     (stroke (width 0) (type default) (color 0 0 0 0))
   )
+  (wire (pts (xy 160.655 72.39) (xy 168.275 72.39))
+    (stroke (width 0) (type default) (color 0 0 0 0))
+  )
   (wire (pts (xy 236.855 72.39) (xy 227.965 72.39))
     (stroke (width 0) (type default) (color 0 0 0 0))
@@
     (stroke (width 0) (type default) (color 0 0 0 0))
   )
-  (wire (pts (xy 160.655 87.63) (xy 168.275 87.63))
-    (stroke (width 0) (type default) (color 0 0 0 0))
-  )
-  (wire (pts (xy 167.005 90.17) (xy 167.005 107.95))
-    (stroke (width 0) (type default) (color 0 0 0 0))
-  )
   (wire (pts (xy 53.975 73.66) (xy 53.975 77.47))
     (stroke (width 0) (type default) (color 0 0 0 0))
@@
     (stroke (width 0) (type default) (color 0 0 0 0))
   )
-  (wire (pts (xy 168.275 87.63) (xy 168.275 97.79))
+  (wire (pts (xy 168.275 72.39) (xy 168.275 97.79))
     (stroke (width 0) (type default) (color 0 0 0 0))
   )
@@
     (stroke (width 0) (type default) (color 0 0 0 0))
   )
-  (wire (pts (xy 160.655 90.17) (xy 167.005 90.17))
+  (wire (pts (xy 167.005 74.93) (xy 160.655 74.93))
     (stroke (width 0) (type default) (color 0 0 0 0))
   )
@@
     (in_bom yes) (on_board yes)
     (property "Reference" "U1" (id 0) (at 195.58 62.865 0))
-    (property "Value" "" (id 1) (at 197.485 66.675 0))
-    (property "Footprint" "" (id 2) (at 208.915 121.92 0)
+    (property "Value" "MAX232" (id 1) (at 197.485 66.675 0))
+    (property "Footprint" "Package_DIP:DIP-16_W7.62mm" (id 2) (at 208.915 121.92 0)
       (effects (font (size 1.27 1.27)) (justify left) hide)
     )
@@
       (effects (font (size 1.524 1.524)))
     )
-    (property "Value" "" (id 1) (at 35.56 61.595 0)
-      (effects (font (size 1.524 1.524)))
-    )
-    (property "Footprint" "" (id 2) (at 36.195 81.28 0)
+    (property "Value" "Jack_LJB0670" (id 1) (at 35.56 61.595 0)
+      (effects (font (size 1.524 1.524)))
+    )
+    (property "Footprint" "D&R_Conn:LJB0670" (id 2) (at 36.195 81.28 0)
       (effects (font (size 1.524 1.524)) hide)
     )
@@
       (effects (font (size 1.524 1.524)))
     )
-    (property "Value" "" (id 1) (at 128.27 60.96 0)
-      (effects (font (size 1.524 1.524)))
-    )
-    (property "Footprint" "" (id 2) (at 173.355 -1.27 0)
+    (property "Value" "Arduino_Uno_Shield" (id 1) (at 128.27 60.96 0)
+      (effects (font (size 1.524 1.524)))
+    )
+    (property "Footprint" "Arduino:Arduino_Uno_Shield_Hat" (id 2) (at 173.355 -1.27 0)
       (effects (font (size 1.524 1.524)) hide)
     )
@@
       (effects (font (size 1.524 1.524)))
     )
-    (property "Value" "" (id 1) (at 35.56 104.14 0)
-      (effects (font (size 1.524 1.524)))
-    )
-    (property "Footprint" "" (id 2) (at 36.195 123.825 0)
+    (property "Value" "Jack_LJB0670" (id 1) (at 35.56 104.14 0)
+      (effects (font (size 1.524 1.524)))
+    )
+    (property "Footprint" "D&R_Conn:LJB0670" (id 2) (at 36.195 123.825 0)
       (effects (font (size 1.524 1.524)) hide)
     )
@@
       (effects (font (size 1.27 1.27)) (justify left))
     )
-    (property "Value" "" (id 1) (at 280.67 123.19 0)
+    (property "Value" "DB9_Male" (id 1) (at 280.67 123.19 0)
       (effects (font (size 1.27 1.27)) (justify left))
     )
-    (property "Footprint" "" (id 2) (at 275.59 123.19 0)
+    (property "Footprint" "Connector_Dsub:DSUB-9_Male_Horizontal_P2.77x2.84mm_EdgePinOffset4.94mm_Housed_MountingHolesOffset7.48mm" (id 2) (at 275.59 123.19 0)
       (effects (font (size 1.27 1.27)) hide)
     )
@@
       (effects (font (size 0.9906 0.9906)) (justify left))
     )
-    (property "Value" "" (id 1) (at 237.363 82.296 0)
-      (effects (font (size 0.9906 0.9906)) (justify left) hide)
-    )
-    (property "Footprint" "" (id 2) (at 237.363 86.106 0)
+    (property "Value" "10U-ALU_16V#CASE_B" (id 1) (at 237.363 82.296 0)
+      (effects (font (size 0.9906 0.9906)) (justify left) hide)
+    )
+    (property "Footprint" "D&R_Passive:C_0805" (id 2) (at 237.363 86.106 0)
       (effects (font (size 0.9906 0.9906)) (justify left) hide)
     )
@@
     (in_bom yes) (on_board yes)
     (property "Reference" "P1" (id 0) (at 243.84 140.335 0))
-    (property "Value" "" (id 1) (at 243.205 142.24 0))
-    (property "Footprint" "" (id 2) (at 243.205 144.78 0))
+    (property "Value" "CONN_02X03" (id 1) (at 243.205 142.24 0))
+    (property "Footprint" "D&R_Conn:HEADER_2x3P" (id 2) (at 243.205 144.78 0))
     (property "Datasheet" "" (id 3) (at 243.205 161.29 0))
     (pin "1")
@@
       (effects (font (size 0.9906 0.9906)) (justify left))
     )
-    (property "Value" "" (id 1) (at 215.519 67.818 0)
-      (effects (font (size 1.524 1.524)) (justify left) hide)
-    )
-    (property "Footprint" "" (id 2) (at 215.265 71.628 0)
+    (property "Value" "100N-X7R_50V#0603" (id 1) (at 215.519 67.818 0)
+      (effects (font (size 1.524 1.524)) (justify left) hide)
+    )
+    (property "Footprint" "D&R_Passive:C_0603" (id 2) (at 215.265 71.628 0)
       (effects (font (size 1.524 1.524)) (justify left) hide)
     )
@@
       (effects (font (size 0.9906 0.9906)) (justify left))
     )
-    (property "Value" "" (id 1) (at 177.673 82.296 0)
-      (effects (font (size 0.9906 0.9906)) (justify left) hide)
-    )
-    (property "Footprint" "" (id 2) (at 177.673 86.106 0)
+    (property "Value" "10U-ALU_16V#CASE_B" (id 1) (at 177.673 82.296 0)
+      (effects (font (size 0.9906 0.9906)) (justify left) hide)
+    )
+    (property "Footprint" "D&R_Passive:C_0805" (id 2) (at 177.673 86.106 0)
       (effects (font (size 0.9906 0.9906)) (justify left) hide)
     )
@@
       (effects (font (size 0.9906 0.9906)) (justify left))
     )
-    (property "Value" "" (id 1) (at 243.967 75.819 0)
-      (effects (font (size 0.9906 0.9906)) (justify left) hide)
-    )
-    (property "Footprint" "" (id 2) (at 243.967 72.009 0)
+    (property "Value" "10U-ALU_16V#CASE_B" (id 1) (at 243.967 75.819 0)
+      (effects (font (size 0.9906 0.9906)) (justify left) hide)
+    )
+    (property "Footprint" "D&R_Passive:C_0805" (id 2) (at 243.967 72.009 0)
       (effects (font (size 0.9906 0.9906)) (justify left) hide)
     )
@@
       (effects (font (size 0.9906 0.9906)) (justify left))
     )
-    (property "Value" "" (id 1) (at 243.967 89.154 0)
-      (effects (font (size 0.9906 0.9906)) (justify left) hide)
-    )
-    (property "Footprint" "" (id 2) (at 243.967 85.344 0)
+    (property "Value" "10U-ALU_16V#CASE_B" (id 1) (at 243.967 89.154 0)
+      (effects (font (size 0.9906 0.9906)) (justify left) hide)
+    )
+    (property "Footprint" "D&R_Passive:C_0805" (id 2) (at 243.967 85.344 0)
       (effects (font (size 0.9906 0.9906)) (justify left) hide)
     )
@@
     (in_bom yes) (on_board yes)
     (property "Reference" "R1" (id 0) (at 57.15 65.405 90))
-    (property "Value" "" (id 1) (at 57.15 69.85 90))
-    (property "Footprint" "" (id 2) (at 57.15 69.088 90)
+    (property "Value" "4k7" (id 1) (at 57.15 69.85 90))
+    (property "Footprint" "D&R_Passive:C_0603" (id 2) (at 57.15 69.088 90)
       (effects (font (size 0.762 0.762)) hide)
     )
@@
     (in_bom yes) (on_board yes)
     (property "Reference" "R2" (id 0) (at 57.15 107.95 90))
-    (property "Value" "" (id 1) (at 57.15 112.395 90))
-    (property "Footprint" "" (id 2) (at 57.15 111.633 90)
+    (property "Value" "4k7" (id 1) (at 57.15 112.395 90))
+    (property "Footprint" "D&R_Passive:C_0603" (id 2) (at 57.15 111.633 90)
       (effects (font (size 0.762 0.762)) hide)
     )
@@
       (effects (font (size 0.9906 0.9906)) (justify right))
     )
-    (property "Value" "" (id 1) (at 65.024 108.712 0)
-      (effects (font (size 1.524 1.524)) (justify left) hide)
-    )
-    (property "Footprint" "" (id 2) (at 64.77 104.902 0)
+    (property "Value" "100N-X7R_50V#0603-D&R_Passive" (id 1) (at 65.024 108.712 0)
+      (effects (font (size 1.524 1.524)) (justify left) hide)
+    )
+    (property "Footprint" "D&R_Passive:C_0603" (id 2) (at 64.77 104.902 0)
       (effects (font (size 1.524 1.524)) (justify left) hide)
     )
@@
       (effects (font (size 0.9906 0.9906)) (justify left))
     )
-    (property "Value" "" (id 1) (at 65.024 65.532 0)
-      (effects (font (size 1.524 1.524)) (justify left) hide)
-    )
-    (property "Footprint" "" (id 2) (at 64.77 61.722 0)
-      (effects (font (size 1.524 1.524)) (justify left) hide)
-    )
+    (property "Value" "100N-X7R_50V#0603-D&R_Passive" (id 1) (at 65.024 65.532 0)
+      (effects (font (size 1.524 1.524)) (justify left) hide)
+    )
+    (property "Footprint" "D&R_Passive:C_0603" (id 2) (at 64.77 61.722 0)
+      (effects (font (size 1.524 1.524)) (justify left) hide)
+    )

Commit message: kicad
Parts:
- removed C5, C7, C8, C9: 10U-ALU_16V#CASE_B, D&R_Passive:C_0805, symbol StartStopTascam-rescue:10U-ALU_16V#CASE_B-D&R_Passive
- removed J1, J2: Jack_LJB0670, D&R_Conn:LJB0670, symbol StartStopTascam-rescue:Jack_LJB0670-D&R_Conn
- added C3, C4, C5, C7: 10U-X5R_25V#1210, D&R_Passive:C_1210, symbol D&R_Passive:10U-X5R_25V#1210
- added C8, C9: 100N-X7R_50V#0603-D&R_Passive, D&R_Passive:C_0603, symbol StartStopTascam-rescue:100N-X7R_50V#0603-D&R_Passive
- added J1, J2: Jack_Stack_LJB0671, D&R_Conn:LJB0671-12, symbol D&R_Conn:Jack_Stack_LJB0671
- added R3, R4: 4k7, D&R_Passive:C_0603, symbol StartStopTascam-rescue:R-D&R_Passive
- J3: value DB9_Male -> (none); symbol Connector:DB9_Male -> StartStopTascam-rescue:DB9_Male
- U1: value MAX232 -> (none); footprint Package_DIP:DIP-16_W7.62mm -> (none)
- XA1: value Arduino_Uno_Shield -> (none); footprint Arduino:Arduino_Uno_Shield_Hat -> (none)
Connections:
- net GND: now also C7.2, C8.1, C9.1, J1.5 (R), J1.7 (R), J2.5 (R), J2.7 (R)
- net VCC: now also C5.1
- net Net-(U1-Pad1): now reaches U1.1 (C1+)
- net Net-(U1-Pad1): now also C3.1
- net Net-(U1-Pad2): now reaches U1.2 (VS+)
- net Net-(U1-Pad2): now also C5.2
- net Net-(U1-Pad3): now reaches U1.3 (C1-)
- net Net-(U1-Pad3): now also C3.2
- net Net-(U1-Pad4): now reaches U1.4 (C2+)
- net Net-(U1-Pad4): now also C4.1
- net Net-(U1-Pad5): now reaches U1.5 (C2-)
- net Net-(U1-Pad5): now also C4.2
- net Net-(U1-Pad6): now reaches U1.6 (VS-)
- net Net-(U1-Pad6): now also C7.1
- net Net-(R1-Pad1): now reaches R1.1
- net Net-(R1-Pad1): now also J1.3 (T)
- net Net-(XA1-PadA0): now reaches XA1.A0
- net Net-(XA1-PadA0): now also C8.2, R3.2
- net Net-(XA1-PadA1): now reaches XA1.A1
- net Net-(XA1-PadA1): now also C9.2, R4.2
- net Net-(XA1-PadA2): now reaches C1.2, R1.2, XA1.A2
- net Net-(XA1-PadA3): now reaches C2.2, R2.2, XA1.A3
- net Net-(R2-Pad1): now reaches R2.1
- net Net-(R2-Pad1): now also J1.1 (T)
- new net: J2.3 (T), R3.1
- new net: J2.1 (T), R4.1
- no-connect marks 48 -> 53
Other:
- moved on the sheet: C2, R2

Commit message: kicad
Parts:
- J3: value (none) -> DB9_Male
- U1: value (none) -> MAX232; footprint (none) -> Package_DIP:DIP-16_W7.62mm
- XA1: value (none) -> Arduino_Uno_Shield; footprint (none) -> Arduino:Arduino_Uno_Shield_Hat
Connections:
- net GND: now also XA1.GND2 (GND)
- no-connect marks 53 -> 52
Changed lines of the file:
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@@
   (junction (at 64.77 67.31) (diameter 0) (color 0 0 0 0)
+  )
+  (junction (at 94.615 113.03) (diameter 0) (color 0 0 0 0)
   )
   (junction (at 64.77 111.76) (diameter 0) (color 0 0 0 0)
@@
   (no_connect (at 94.615 74.93))
   (no_connect (at 94.615 115.57))
-  (no_connect (at 94.615 110.49))
   (no_connect (at 94.615 107.95))
   (no_connect (at 160.655 107.95))
@@
     (stroke (width 0) (type default) (color 0 0 0 0))
   )
+  (wire (pts (xy 94.615 110.49) (xy 94.615 113.03))
+    (stroke (width 0) (type default) (color 0 0 0 0))
+  )
   (wire (pts (xy 51.435 113.03) (xy 51.435 111.76))
     (stroke (width 0) (type default) (color 0 0 0 0))
@@
     (in_bom yes) (on_board yes)
     (property "Reference" "U1" (id 0) (at 195.58 62.865 0))
-    (property "Value" "" (id 1) (at 197.485 66.675 0))
-    (property "Footprint" "" (id 2) (at 208.915 121.92 0)
+    (property "Value" "MAX232" (id 1) (at 197.485 66.675 0))
+    (property "Footprint" "Package_DIP:DIP-16_W7.62mm" (id 2) (at 208.915 121.92 0)
       (effects (font (size 1.27 1.27)) (justify left) hide)
     )
@@
       (effects (font (size 1.524 1.524)))
     )
-    (property "Value" "" (id 1) (at 128.27 60.96 0)
-      (effects (font (size 1.524 1.524)))
-    )
-    (property "Footprint" "" (id 2) (at 173.355 -1.27 0)
+    (property "Value" "Arduino_Uno_Shield" (id 1) (at 128.27 60.96 0)
+      (effects (font (size 1.524 1.524)))
+    )
+    (property "Footprint" "Arduino:Arduino_Uno_Shield_Hat" (id 2) (at 173.355 -1.27 0)
       (effects (font (size 1.524 1.524)) hide)
     )
@@
       (effects (font (size 1.27 1.27)) (justify left))
     )
-    (property "Value" "" (id 1) (at 280.67 123.19 0)
+    (property "Value" "DB9_Male" (id 1) (at 280.67 123.19 0)
       (effects (font (size 1.27 1.27)) (justify left))
     )
@@
       (effects (font (size 1.27 1.27)) hide)
     )
-    (property "Value" "" (id 1) (at 244.475 104.14 0))
+    (property "Value" "GND" (id 1) (at 244.475 104.14 0))
     (property "Footprint" "" (id 2) (at 244.475 99.06 0)
       (effects (font (size 1.27 1.27)) hide)
@@
       (effects (font (size 1.27 1.27)) hide)
     )
-    (property "Value" "" (id 1) (at 67.31 123.1901 0)
+    (property "Value" "GND" (id 1) (at 67.31 123.1901 0)
       (effects (font (size 1.27 1.27)) (justify right))
     )

Commit message: Kicad
Kicad
Parts:
- added D1: TSAL4400, LED_THT:LED_D3.0mm_IRBlack, symbol LED:TSAL4400
- added R5: 470R#0603, D&R_Passive:R_0603, symbol D&R_Passive:470R#0603
Connections:
- net VCC: now also R5.1
- net at U1.11 (T1IN): now also XA1.D3 (D3_INT1); no longer XA1.D4
- net at U1.12 (R1OUT): now also XA1.D4; no longer XA1.D5
- net at XA1.D2 (D2_INT0): now also D1.1 (K)
- new net: D1.2 (A), R5.2
- no-connect marks 52 -> 51
